File: board/board.kicad_pcb (KiCad board)
At the start: 2 copper layers, 21 x 13 mm, 1 part

Commit message: initial
Parts:
- added C1: 100nF, Capacitor_SMD:C_0603_1608Metric, F.Cu at (149.5, 92.8)
- added C2: 100nF, Capacitor_SMD:C_0603_1608Metric, F.Cu at (151.0, 92.8)
- added J1: 002_SPI, on_edge:on_edge_2x05_device, F.Cu at (140.0, 96.5)
- added J2: 007_ADC, on_edge:on_edge_2x05_host, F.Cu at (161.0, 96.5)
- added U1: ADS1120IRVAR, b110:QFN50P350X350X100-17N, F.Cu at (150.5, 97.0)
- LOGO1: moved to B.Cu
- moved LOGO1 0.85 mm to (150.6, 98.4), turned to 180 degrees
Routing:
- net +3.3V: track 0.00 -> 32.0 mm, vias 0 -> 1
- net GND: track 0.00 -> 31.0 mm, vias 0 -> 3
- net Net-(J1-Pad10): track 0.00 -> 16.7 mm
- net /adc/AD3: track 0.00 -> 12.4 mm, vias 0 -> 1
- net /adc/DRDY: track 0.00 -> 11.6 mm, vias 0 -> 2
- net /adc/CS: track 0.00 -> 9.85 mm, vias 0 -> 1
- net /adc/AD0: track 0.00 -> 8.38 mm
- net /adc/AD2: track 0.00 -> 8.24 mm
- net /adc/AD1: track 0.00 -> 7.40 mm
- net /adc/MOSI: track 0.00 -> 7.40 mm
- net /adc/SCLK: track 0.00 -> 7.36 mm
- net /adc/MISO: track 0.00 -> 6.58 mm, vias 0 -> 2
Other:
- outline, holes or cut-outs redrawn
- board text added: "osf.002"
- board text added: "osf.007"
- board text added: "osf.b110.v1.0"
