File: board/board.kicad_pcb (KiCad board)
At the start: 2 copper layers, 21 x 13 mm, 6 parts, among them J1 002_SPI, J2 007_ADC, U1 ADS1120IRVAR

Commit message: added jlc production files and some cosmetic changes
Connections:
- net Net-(J1-Pad10) renamed /5V
